File: Gateway/PCB/PCB_gateway.kicad_sch (KiCad schematic)
At the start: 37 parts, among them J1 USB4215-03-A_REVA, J2 Conn_01x06_Pin, J3 Conn_01x04_Pin, J4 Conn_01x04_Pin, U1 ESP32-C3-WROOM-02U-N4, U2 BME680, U4 AMS1117-3.3

Commit message: Add files via upload
Parts:
- added R12, R13: 0, Resistor_SMD:R_0805_2012Metric_Pad1.20x1.40mm_HandSolder, symbol Device:R
- renumbered S2 to BOOT1, S1 to EN1, D1 to LED1, D2 to POWER1
Connections:
- net D+: now also R13.1; no longer J1.A6 (DP1), J1.B6 (DP2)
- net D-: now also R12.2; no longer J1.A7 (DN1), J1.B7 (DN2)
- net RX: now also J3.3 (Pin_3); no longer J3.2 (Pin_2)
- net TX: now also J3.2 (Pin_2); no longer J3.3 (Pin_3)
- new net: J1.A6 (DP1), J1.B6 (DP2), R13.2
- new net: J1.A7 (DN1), J1.B7 (DN2), R12.1
Changed lines of the file:
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@@
 	)
 	(junction
+		(at 71.12 168.91)
+		(diameter 0)
+		(color 0 0 0 0)
+	)
+	(junction
 		(at 107.95 69.85)
 		(diameter 0)
@@
 	)
 	(junction
+		(at 35.56 166.37)
+		(diameter 0)
+		(color 0 0 0 0)
+	)
+	(junction
 		(at 93.98 163.83)
 		(diameter 0)
@@
 	(wire
 		(pts
-			(xy 71.12 167.64) (xy 71.12 170.18)
+			(xy 71.12 167.64) (xy 71.12 168.91)
 		)
 		(stroke
@@
 	(wire
 		(pts
+			(xy 71.12 168.91) (xy 71.12 170.18)
+		)
+		(stroke
+			(width 0)
+			(type default)
+		)
+	)
+	(wire
+		(pts
 			(xy 129.54 46.99) (xy 123.19 46.99)
 		)
@@
 	(wire
 		(pts
-			(xy 35.56 165.1) (xy 35.56 167.64)
+			(xy 35.56 165.1) (xy 35.56 166.37)
 		)
 		(stroke
@@
 	(wire
 		(pts
+			(xy 35.56 166.37) (xy 35.56 167.64)
+		)
+		(stroke
+			(width 0)
+			(type default)
+		)
+	)
+	(wire
+		(pts
 			(xy 170.18 95.25) (xy 170.18 96.52)
 		)
@@
 		)
 	)
-	(global_label "D+"
-		(shape input)
-		(at 35.56 166.37 180)
-		(fields_autoplaced yes)
-		(effects
-			(font
-				(size 1.27 1.27)
-			)
-			(justify right)
-		)
-		(property "Intersheetrefs" "${INTERSHEET_REFS}"
-			(at 29.7324 166.37 0)
-			(effects
-				(font
-					(size 1.27 1.27)
-				)
-				(justify right)
-				(hide yes)
-			)
-		)
-	)
 	(global_label "SDA"
 		(shape input)
@@
 		)
 	)
-	(global_label "TX"
+	(global_label "RX"
 		(shape input)
 		(at 234.95 144.78 0)
@@
 		)
 		(property "Intersheetrefs" "${INTERSHEET_REFS}"
-			(at 240.1123 144.78 0)
+			(at 240.4147 144.78 0)
 			(effects
 				(font
@@
 		)
 	)
+	(global_label "D+"
+		(shape input)
+		(at 27.94 166.37 180)
+		(fields_autoplaced yes)
+		(effects
+			(font
+				(size 1.27 1.27)
+			)
+			(justify right)
+		)
+		(property "Intersheetrefs" "${INTERSHEET_REFS}"
+			(at 22.1124 166.37 0)
+			(effects
+				(font
+					(size 1.27 1.27)
+				)
+				(justify right)
+				(hide yes)
+			)
+		)
+	)
 	(global_label "GPIO1"
 		(shape input)
@@
 	(global_label "D-"
 		(shape input)
+		(at 78.74 168.91 0)
+		(fields_autoplaced yes)
+		(effects
+			(font
+				(size 1.27 1.27)
+			)
+			(justify left)
+		)
+		(property "Intersheetrefs" "${INTERSHEET_REFS}"
+			(at 84.5676 168.91 0)
+			(effects
+				(font
+					(size 1.27 1.27)
+				)
+				(justify left)
+				(hide yes)
+			)
+		)
+	)
+	(global_label "D-"
+		(shape input)
 		(at 107.95 54.61 0)
 		(fields_autoplaced yes)
@@
 		)
 	)
-	(global_label "D-"
-		(shape input)
-		(at 71.12 168.91 0)
-		(fields_autoplaced yes)
-		(effects
-			(font
-				(size 1.27 1.27)
-			)
-			(justify left)
-		)
-		(property "Intersheetrefs" "${INTERSHEET_REFS}"
-			(at 76.9476 168.91 0)
-			(effects
-				(font
-					(size 1.27 1.27)
-				)
-				(justify left)
-				(hide yes)
-			)
-		)
-	)
 	(global_label "GPIO3"
 		(shape input)
@@
 		)
 	)
-	(global_label "RX"
+	(global_label "TX"
 		(shape input)
 		(at 234.95 142.24 0)
@@
 		)
 		(property "Intersheetrefs" "${INTERSHEET_REFS}"
-			(at 240.4147 142.24 0)
+			(at 240.1123 142.24 0)
 			(effects
 				(font
@@
 		(on_board yes)
 		(dnp no)
-		(fields_autoplaced yes)
-		(property "Reference" "D2"
-			(at 259.3975 85.09 0)
+		(property "Reference" "POWER1"
+			(at 257.81 86.614 0)
 			(effects
 				(font
@@
 		)
 		(property "Value" "LED"
-			(at 259.3975 87.63 0)
+			(at 257.81 89.154 0)
 			(effects
 				(font
@@
 			(project "PCB_gateway"
 				(path "/42271d13-3797-4ead-80a1-7080d9d67565"
-					(reference "D2")
+					(reference "POWER1")
 					(unit 1)
 				)
@@
 	)
 	(symbol
+		(lib_id "Device:R")
+		(at 74.93 168.91 90)
+		(unit 1)
+		(exclude_from_sim no)
+		(in_bom yes)
+		(on_board yes)
+		(dnp no)
+		(property "Reference" "R12"
+			(at 74.93 164.084 90)
+			(effects
+				(font
+					(size 1.27 1.27)
+				)
+			)
+		)
+		(property "Value" "0"
+			(at 74.93 166.624 90)
+			(effects
+				(font
+					(size 1.27 1.27)
+				)
+			)
+		)
+		(property "Footprint" "Resistor_SMD:R_0805_2012Metric_Pad1.20x1.40mm_HandSolder"
+			(at 74.93 170.688 90)
+			(effects
+				(font
+					(size 1.27 1.27)
+				)
+				(hide yes)
+			)
+		)
+		(property "Datasheet" "~"
+			(at 74.93 168.91 0)
+			(effects
+				(font
+					(size 1.27 1.27)
+				)
+				(hide yes)
+			)
+		)
+		(property "Description" "Resistor"
+			(at 74.93 168.91 0)
+			(effects
+				(font
+					(size 1.27 1.27)
+				)
+				(hide yes)
+			)
+		)
+		(pin "1"
+		)
+		(pin "2"
+		)
+		(instances
+			(project ""
+				(path "/42271d13-3797-4ead-80a1-7080d9d67565"
+					(reference "R12")
+					(unit 1)
+				)
+			)
+		)
+	)
+	(symbol
 		(lib_id "power:+3.3V")
 		(at 170.18 68.58 0)
@@
 		(on_board yes)
 		(dnp no)
-		(property "Reference" "S1"
+		(property "Reference" "EN1"
 			(at 176.53 87.63 90)
 			(effects
@@
 			(project ""
 				(path "/42271d13-3797-4ead-80a1-7080d9d67565"
-					(reference "S1")
+					(reference "EN1")
 					(unit 1)
 				)
@@
 		(on_board yes)
 		(dnp no)
-		(fields_autoplaced yes)
 		(property "Reference" "#FLG02"
 			(at 33.655 160.02 0)
@@
 		)
 		(property "Value" "PWR_FLAG"
-			(at 31.75 160.0199 90)
+			(at 34.798 157.48 90)
 			(effects
 				(font
@@
 		(on_board yes)
 		(dnp no)
-		(fields_autoplaced yes)
-		(property "Reference" "D1"
-			(at 259.3975 71.12 0)
+		(property "Reference" "LED1"
+			(at 257.81 72.644 0)
 			(effects
 				(font
@@
 		)
 		(property "Value" "LED"
-			(at 259.3975 73.66 0)
+			(at 257.81 75.184 0)
 			(effects
 				(font
@@
 			(project ""
 				(path "/42271d13-3797-4ead-80a1-7080d9d67565"
-					(reference "D1")
+					(reference "LED1")
 					(unit 1)
 				)
@@
 		(on_board yes)
 		(dnp no)
-		(property "Reference" "S2"
-			(at 201.93 87.63 90)
+		(property "Reference" "BOOT1"
+			(at 202.692 87.63 90)
 			(effects
 				(font
@@
 			(project "PCB_gateway"
 				(path "/42271d13-3797-4ead-80a1-7080d9d67565"
-					(reference "S2")
+					(reference "BOOT1")
 					(unit 1)
 				)
@@
 					(unit 1)
 				)
+			)
+		)
+	)
+	(symbol
+		(lib_id "Device:R")
+		(at 31.75 166.37 90)
+		(unit 1)
+		(exclude_from_sim no)
+		(in_bom yes)
+		(on_board yes)
+		(dnp no)
+		(property "Reference" "R13"
+			(at 31.75 162.052 90)
+			(effects
+				(font
+					(size 1.27 1.27)
+				)
+			)
+		)
+		(property "Value" "0"
+			(at 31.75 164.084 90)
+			(effects
+				(font
+					(size 1.27 1.27)
+				)
+			)
+		)
+		(property "Footprint" "Resistor_SMD:R_0805_2012Metric_Pad1.20x1.40mm_HandSolder"
+			(at 31.75 168.148 90)
+			(effects
+				(font
+					(size 1.27 1.27)
+				)
+				(hide yes)
+			)
+		)
+		(property "Datasheet" "~"
+			(at 31.75 166.37 0)
+			(effects
+				(font
+					(size 1.27 1.27)
+				)
+				(hide yes)
+			)
+		)
+		(property "Description" "Resistor"
+			(at 31.75 166.37 0)
+			(effects
+				(font
+					(size 1.27 1.27)
+				)
+				(hide yes)
+			)
+		)
+		(pin "1"
+		)
+		(pin "2"
+		)
+		(instances
+			(project "PCB_gateway"
+				(path "/42271d13-3797-4ead-80a1-7080d9d67565"
+					(reference "R13")
+					(unit 1)
+				)
